File: schematic.sch (EAGLE design)
At the start: 8 parts, among them IC1 DS1820

Commit message: schematic update and picture of schematic
Parts:
- C1, C2: value (none) -> 100uF
- U$1: value V_REG_LD1117VXX -> LD1117V33
- U1: value (none) -> RHT03
- renumbered D1 to J1, IC1 to U2
Other:
- note added: "5-15VDC"
